Commit message: added slam

File: robot_dd/description/lidar.xacro (robot description, xacro)
@@ -26,5 +26,5 @@
         <sensor name="laser" type="ray">
             <pose> 0 0 0 0 0 0 </pose>
-            <visualize>false</visualize>
+            <visualize>true</visualize>
             <update_rate>10</update_rate>
             <ray>

File: robot_dd/description/robot.urdf.xacro (robot description, xacro)
@@ -12,4 +12,4 @@
   <!-- <xacro:include filename="camera.xacro"/> -->
   <!-- Depth Camera -->
-  <xacro:include filename="depth_camera.xacro"/>
+  <!-- <xacro:include filename="depth_camera.xacro"/> -->
 </robot>

File: robot_dd/description/robot_core.xacro (robot description, xacro)
@@ -4,6 +4,12 @@
   <xacro:include filename="inertial_macro.xacro"/>
   <!-- BASE LINK -->
-  <link name="base_link">
-  </link>
+  <link name="base_link"/>
+  <!-- BASE FOOTPRINT -->
+  <joint name="base_footprint_joint" type="fixed">
+    <parent link="base_link"/>
+    <child link="base_footprint"/>
+    <origin xyz="0.0 0.0 0.0" rpy="0.0 0.0 0.0"/>
+  </joint>
+  <link name="base_footprint"/>
   <!-- CHASSIS LINK-->
   <joint name="chassis_link" type="fixed">
