Commit message: added gazebo control & ros2 control

File: robot_dd/description/material.xacro (robot description, xacro)
@@ -13,3 +13,6 @@
     <color rgba="0.2 0.2 1 1" />
   </material>
+  <material name="red">
+    <color rgba="1 0 0 1" />
+  </material>
 </robot>

File: robot_dd/description/robot.urdf.xacro (robot description, xacro)
@@ -1,4 +1,15 @@
 <?xml version="1.0"?>
 <robot xmlns:xacro="http://www.ros.org/wiki/xacro" name="robot_dd">
+  <!-- ROBOT URDF-->
   <xacro:include filename="robot_core.xacro"/>
+  <!-- Gazebo Controller -->
+  <!-- <xacro:include filename="gazebo_control.xacro"/> -->
+  <!-- ROS2 Control -->
+  <xacro:include filename="ros2_control.xacro"/>
+  <!-- Lidar 2D -->
+  <xacro:include filename="lidar.xacro"/>
+  <!-- Camera -->
+  <!-- <xacro:include filename="camera.xacro"/> -->
+  <!-- Depth Camera -->
+  <xacro:include filename="depth_camera.xacro"/>
 </robot>

File: robot_dd/description/robot_core.xacro (robot description, xacro)
@@ -14,5 +14,5 @@
   <link name="chassis">
     <visual>
-      <origin xyz="0.15 0.0 0.075" rpy="0.0 0.0 0.0"/>
+      <origin xyz="0.15 0.0 0.075"/>
       <geometry>
         <box size="0.3 0.3 0.15"/>
@@ -21,5 +21,5 @@
     </visual>
     <collision>
-      <origin xyz="0.15 0.0 0.075" rpy="0.0 0.0 0.0"/>
+      <origin xyz="0.15 0.0 0.075"/>
       <geometry>
         <box size="0.3 0.3 0.15"/>
@@ -27,7 +27,10 @@
     </collision>
     <xacro:inertial_box mass="0.5" x="0.3" y="0.3" z="0.15">
-      <origin xyz="0.0 0.0 0.0" rpy="0.0 0.0 0.0"/>
+      <origin xyz="0.15 0.0 0.075" rpy="0.0 0.0 0.0"/>
     </xacro:inertial_box>
   </link>
+  <gazebo reference="chassis">
+    <material>Gazebo/White</material>
+  </gazebo>
   <!-- LEFT WHEEL LINK-->
   <joint name="left_wheel_joint" type="continuous">
@@ -53,4 +56,7 @@
     </xacro:inertial_cylinder>
   </link>
+  <gazebo reference="left_wheel">
+    <material>Gazebo/Blue</material>
+  </gazebo>
   <!-- RIGHT WHEEL LINK-->
   <joint name="right_wheel_joint" type="continuous">
@@ -76,11 +82,14 @@
     </xacro:inertial_cylinder>
   </link>
+  <gazebo reference="right_wheel">
+    <material>Gazebo/Blue</material>
+  </gazebo>
   <!-- CASTOR WHEEL JOINT -->
   <joint name="caster_wheel_joint" type="fixed">
     <parent link="chassis"/>
-    <child link="castor_wheel"/>
+    <child link="caster_wheel"/>
     <origin xyz="0.24 0.0 0.0" rpy="0.0 0.0 0.0"/>
   </joint>
-  <link name="castor_wheel">
+  <link name="caster_wheel">
     <visual>
       <geometry>
@@ -98,3 +107,8 @@
     </xacro:inertial_sphere>
   </link>
+  <gazebo reference="caster_wheel">
+    <material>Gazebo/Black</material>
+    <mu1 value="0.001"/>
+    <mu2 value="0.001"/>
+  </gazebo>
 </robot>

Commit message: changed robot model and launch files

File: robot_dd/description/material.xacro (robot description, xacro)
@@ -1,18 +1,33 @@
 <?xml version="1.0"?>
 <robot xmlns:xacro="http://www.ros.org/wiki/xacro" name="robot_dd">
-  <material name="white">
-    <color rgba="1 1 1 1" />
+  <material name="black">
+    <color rgba="0.0 0.0 0.0 1.0"/>
   </material>
-  <material name="black">
-    <color rgba="0 0 0 1" />
+  <material name="dark">
+    <color rgba="0.3 0.3 0.3 1.0"/>
+  </material>
+  <material name="light_black">
+    <color rgba="0.4 0.4 0.4 1.0"/>
+  </material>
+  <material name="blue">
+    <color rgba="0.0 0.0 0.8 1.0"/>
+  </material>
+  <material name="green">
+    <color rgba="0.0 0.8 0.0 1.0"/>
+  </material>
+  <material name="grey">
+    <color rgba="0.5 0.5 0.5 1.0"/>
   </material>
   <material name="orange">
-    <color rgba="1 0.3 0.1 1" />
+    <color rgba="1.0 0.4235 0.0392 1.0"/>
   </material>
-  <material name="blue">
-    <color rgba="0.2 0.2 1 1" />
+  <material name="brown">
+    <color rgba="0.8706 0.8118 0.7647 1.0"/>
   </material>
   <material name="red">
-    <color rgba="1 0 0 1" />
+    <color rgba="0.8 0.0 0.0 1.0"/>
+  </material>
+  <material name="white">
+    <color rgba="1.0 1.0 1.0 1.0"/>
   </material>
 </robot>
