Commit message: restructured urdf & added gazebo colors

File: questbot_description/urdf/robot/materials.xacro (robot description, xacro)
@@ -1,12 +1,7 @@
 <?xml version="1.0"?>
 <robot xmlns:xacro="http://www.ros.org/wiki/xacro" name="questbot_2wd">
+  <!-- Rviz Colours -->
   <material name="black">
     <color rgba="0.0 0.0 0.0 1.0"/>
-  </material>
-  <material name="dark">
-    <color rgba="0.3 0.3 0.3 1.0"/>
-  </material>
-  <material name="light_black">
-    <color rgba="0.4 0.4 0.4 1.0"/>
   </material>
   <material name="blue">
@@ -28,6 +23,6 @@
     <color rgba="0.8 0.0 0.0 1.0"/>
   </material>
-  <material name="white">
-    <color rgba="1.0 1.0 1.0 1.0"/>
+  <material name="cyan">
+    <color rgba="0 1.0 1.0 1.0"/>
   </material>
 </robot>

File: questbot_description/urdf/robot/robot.model.xacro (robot description, xacro)
@@ -2,10 +2,12 @@
 <robot xmlns:xacro="http://www.ros.org/wiki/xacro" >
     <!-- Including files -->
-    <!-- Include material colors -->
-    <xacro:include filename="material.xacro"/>
+    <!-- Include rviz material colors -->
+    <xacro:include filename="materials.xacro"/>
+    <!-- Include gazebo material colors -->
+    <xacro:include filename="materials.gazebo.xacro"/>
     <!-- Include inertial macros -->
-    <xacro:include filename="macros/inertial.xacro"/>
+    <xacro:include filename="inertial_macro.xacro"/>
     <!-- Include wheel macros -->
-    <xacro:include filename="macros/wheel.xacro"/>
+    <xacro:include filename="wheel_macro.xacro"/>
     <!-- Define robot constants -->
     <!-- Robot base constants -->
@@ -27,7 +29,5 @@
             <box size="${base_length} ${base_width} ${base_height}"/>
         </geometry>
-        <material name="Cyan">
-            <color rgba="0 1.0 1.0 1.0"/>
-        </material>
+        <material name="blue"/>
         </visual>
         <collision>
@@ -51,7 +51,5 @@
             <sphere radius="${(wheel_radius+wheel_zoff-(base_height/2))}"/>
         </geometry>
-        <material name="Cyan">
-            <color rgba="0 1.0 1.0 1.0"/>
-        </material>
+        <material name="grey"/>
         </visual>
         <collision>

File: questbot_description/urdf/robot/wheel_macro.xacro (robot description, xacro)
@@ -9,7 +9,5 @@
                 <cylinder radius="${wheel_radius}" length="${wheel_width}"/>
             </geometry>
-            <material name="Gray">
-            <color rgba="0.5 0.5 0.5 1.0"/>
-            </material>
+            <material name="grey"/>
         </visual>
         <collision>
