Commit message: added till gazebo classic launch file

File: questbot_description/urdf/gazebo.urdf.xacro (robot description, xacro)
@@ -1,17 +1,23 @@
 <?xml version="1.0"?>
 <robot xmlns:xacro="http://www.ros.org/wiki/xacro">
+    <xacro:property name="use_gazebo" value="1"/>
+    <xacro:property name="use_gzsim" value="0"/>
     <!-- Classic Gazebo -->
-    <!-- Controller -->
-    <xacro:include filename="control/gazebo_control.xacro"/>
-    <!-- IMU gazebo plugin -->
-    <xacro:include filename="sensors/gazebo_imu.xacro"/>
-    <!-- Lidar 2D -->
-    <xacro:include filename="sensors/gazebo_lidar.xacro"/>
-    <!-- Camera -->
-    <!-- <xacro:include filename="sensors/gazebo_camera.xacro"/> -->
-    <!-- Depth Camera -->
-    <!-- <xacro:include filename="sensors/gazebo_depth_camera.xacro"/> -->
-    <!-- Gazebo Sim Plugins-->
-    <!-- Controller -->
-    <!-- <xacro:include filename="control/gazebo2_control.xacro"/> -->
+    <xacro:if value="$(arg use_gazebo)">
+        <!-- Controller -->
+        <xacro:include filename="control/gazebo_control.xacro"/>
+        <!-- IMU gazebo plugin -->
+        <xacro:include filename="sensors/gazebo_imu.xacro"/>
+        <!-- Lidar 2D -->
+        <xacro:include filename="sensors/gazebo_lidar.xacro"/>
+        <!-- Camera -->
+        <!-- <xacro:include filename="sensors/gazebo_camera.xacro"/> -->
+        <!-- Depth Camera -->
+        <!-- <xacro:include filename="sensors/gazebo_depth_camera.xacro"/> -->
+    </xacro:if>
+    <!-- Gazebo Sim Plugins -->
+    <xacro:if value="$(arg use_gzsim)">
+        <!-- Controller -->
+        <xacro:include filename="control/gzsim_control.xacro"/>
+    </xacro:if>
 </robot>
