Commit message: changed overall structure

File: questbot_description/urdf/body.urdf.xacro (robot description, xacro)
@@ -2,9 +2,8 @@
 <robot xmlns:xacro="http://www.ros.org/wiki/xacro" >
     <!-- Including files -->
-    <!-- Include inertial macros -->
-    <xacro:include filename="inertial_macros.xacro"/>
-    <!-- Visual -->
-    <!-- Include rviz material colors -->
-    <xacro:include filename="materials.xacro"/>
+    <!-- Inertial -->
+    <xacro:include filename="macro/inertial.xacro"/>
+    <!-- Wheel -->
+    <xacro:include filename="macro/wheel.xacro"/>
     <!-- Define robot constants -->
     <!-- Robot base constants -->
@@ -23,8 +22,10 @@
     <link name="base_link">
         <visual>
-        <geometry>
-            <box size="${base_length} ${base_width} ${base_height}"/>
-        </geometry>
-        <material name="cyan"/>
+            <geometry>
+                <box size="${base_length} ${base_width} ${base_height}"/>
+            </geometry>
+            <material name="turquoise">
+                <color rgba="0 1.0 1.0 1.0"/>
+            </material>
         </visual>
         <collision>
@@ -35,4 +36,7 @@
         <xacro:box_inertia mass="15" width="${base_width}" length="${base_length}" height="${base_height}"/>
     </link>
+    <gazebo reference="base_link">
+        <material>Gazebo/Turquoise</material>
+    </gazebo>
     <!-- Robot Footprint -->
     <link name="base_footprint"/>
@@ -45,8 +49,10 @@
     <link name="front_caster">
         <visual>
-        <geometry>
-            <sphere radius="${(wheel_radius+wheel_zoff-(base_height/2))}"/>
-        </geometry>
-        <material name="grey"/>
+            <geometry>
+                <sphere radius="${(wheel_radius+wheel_zoff-(base_height/2))}"/>
+            </geometry>
+            <material name="grey">
+                <color rgba="0.5 0.5 0.5 1.0"/>
+            </material>
         </visual>
         <collision>
@@ -63,3 +69,11 @@
         <origin xyz="${caster_xoff} 0.0 ${-(base_height/2)}" rpy="0 0 0"/>
     </joint>
+    <gazebo reference="front_caster">
+        <material>Gazebo/Grey</material>
+        <mu1 value="0.001"/>
+        <mu2 value="0.001"/>
+    </gazebo>
+    <!-- Wheels -->
+    <xacro:wheel prefix="left_wheel" x_reflect="-1" y_reflect="1" />
+    <xacro:wheel prefix="right_wheel" x_reflect="-1" y_reflect="-1" />
 </robot>

File: questbot_description/urdf/gazebo.urdf.xacro (robot description, xacro)
@@ -1,5 +1,5 @@
 <?xml version="1.0"?>
 <robot xmlns:xacro="http://www.ros.org/wiki/xacro">
-    <!-- Classic Gazebo Plugins -->
+    <!-- Classic Gazebo -->
     <!-- Controller -->
     <xacro:include filename="control/gazebo_control.xacro"/>
@@ -15,17 +15,3 @@
     <!-- Controller -->
     <!-- <xacro:include filename="control/gazebo2_control.xacro"/> -->
-    <gazebo reference="base_link">
-        <material>Gazebo/Turquoise</material>
-    </gazebo>
-     <gazebo reference="front_caster">
-        <material>Gazebo/Grey</material>
-        <mu1 value="0.001"/>
-        <mu2 value="0.001"/>
-    </gazebo>
-    <gazebo reference="left_wheel_link">
-        <material>Gazebo/Grey</material>
-    </gazebo>
-    <gazebo reference="right_wheel_link">
-        <material>Gazebo/Grey</material>
-    </gazebo>
 </robot>

File: questbot_description/urdf/robot.urdf.xacro (robot description, xacro)
@@ -2,7 +2,5 @@
 <robot xmlns:xacro="http://www.ros.org/wiki/xacro" name="questbot_2wd">
     <!-- Robot Body-->
-    <xacro:include filename="parts/body.urdf.xacro"/>
-    <!-- Robot Wheels -->
-    <xacro:include filename="parts/wheel.xacro"/>
+    <xacro:include filename="body.urdf.xacro"/>
     <!-- Gazebo Definitions -->
     <xacro:include filename="gazebo.urdf.xacro"/>

File: questbot_description/urdf/sensors/gazebo_depth_camera.xacro (robot description, xacro)
@@ -21,13 +21,13 @@
     </link>
     <joint name="camera_joint" type="fixed">
-    <parent link="base_link"/>
-    <child link="camera_link"/>
-    <origin xyz="0.215 0 0.05" rpy="0 0 0"/>
+        <parent link="base_link"/>
+        <child link="camera_link"/>
+        <origin xyz="0.215 0 0.05" rpy="0 0 0"/>
     </joint>
     <link name="camera_depth_frame"/>
     <joint name="camera_depth_joint" type="fixed">
-    <origin xyz="0 0 0" rpy="${-pi/2} 0 ${-pi/2}"/>
-    <parent link="camera_link"/>
-    <child link="camera_depth_frame"/>
+        <origin xyz="0 0 0" rpy="${-pi/2} 0 ${-pi/2}"/>
+        <parent link="camera_link"/>
+        <child link="camera_depth_frame"/>
     </joint>
     <gazebo reference="camera_link">

File: questbot_description/urdf/sensors/gazebo_imu.xacro (robot description, xacro)
@@ -6,5 +6,7 @@
                 <box size="0.1 0.1 0.1"/>
             </geometry>
-            <material name="lightblue"/>
+            <material name="skyblue">
+                <color rgba="0.529 0.808 0.922 1.0"/>
+            </material>
         </visual>
         <collision>
@@ -20,4 +22,8 @@
         <origin xyz="0 0 0.01"/>
     </joint>
+    <gazebo reference="imu_link">
+        <material>Gazebo/SkyBlue</material>
+    </gazebo>
+    <!-- Gazebo Plugin -->
     <gazebo reference="imu_link">
         <sensor name="imu_sensor" type="imu">
@@ -82,5 +88,5 @@
             </linear_acceleration>
         </imu>
-    </sensor>
-</gazebo>
+        </sensor>
+    </gazebo>
 </robot>
