Commit message: linted xml & python files

File: questbot_description/urdf/body.urdf.xacro (robot description, xacro)
@@ -1,38 +1,39 @@
 <?xml version="1.0"?>
-<robot xmlns:xacro="http://www.ros.org/wiki/xacro" >
+<robot xmlns:xacro="http://www.ros.org/wiki/xacro">
     <!-- Including files -->
     <!-- Inertial -->
-    <xacro:include filename="macro/inertial.xacro"/>
+    <xacro:include filename="macro/inertial.xacro" />
     <!-- Wheel -->
-    <xacro:include filename="macro/wheel.xacro"/>
+    <xacro:include filename="macro/wheel.xacro" />
     <!-- Define robot constants -->
     <!-- Robot base constants -->
-    <xacro:property name="base_width" value="0.31"/>
-    <xacro:property name="base_length" value="0.42"/>
-    <xacro:property name="base_height" value="0.18"/>
+    <xacro:property name="base_width" value="0.31" />
+    <xacro:property name="base_length" value="0.42" />
+    <xacro:property name="base_height" value="0.18" />
     <!-- Robot wheels constants -->
-    <xacro:property name="wheel_radius" value="0.10"/>
-    <xacro:property name="wheel_width" value="0.04"/>
-    <xacro:property name="wheel_ygap" value="0.025"/>
-    <xacro:property name="wheel_zoff" value="0.05"/>
-    <xacro:property name="wheel_xoff" value="0.12"/>
+    <xacro:property name="wheel_radius" value="0.10" />
+    <xacro:property name="wheel_width" value="0.04" />
+    <xacro:property name="wheel_ygap" value="0.025" />
+    <xacro:property name="wheel_zoff" value="0.05" />
+    <xacro:property name="wheel_xoff" value="0.12" />
     <!-- Castor wheels constats -->
-    <xacro:property name="caster_xoff" value="0.14"/>
+    <xacro:property name="caster_xoff" value="0.14" />
     <!-- Robot Base -->
     <link name="base_link">
         <visual>
             <geometry>
-                <box size="${base_length} ${base_width} ${base_height}"/>
+                <box size="${base_length} ${base_width} ${base_height}" />
             </geometry>
             <material name="turquoise">
-                <color rgba="0 1.0 1.0 1.0"/>
+                <color rgba="0 1.0 1.0 1.0" />
             </material>
         </visual>
         <collision>
             <geometry>
-                <box size="${base_length} ${base_width} ${base_height}"/>
+                <box size="${base_length} ${base_width} ${base_height}" />
             </geometry>
         </collision>
-        <xacro:box_inertia mass="15" width="${base_width}" length="${base_length}" height="${base_height}"/>
+        <xacro:box_inertia mass="15" width="${base_width}" length="${base_length}"
+            height="${base_height}" />
     </link>
     <gazebo reference="base_link">
@@ -40,9 +41,9 @@
     </gazebo>
     <!-- Robot Footprint -->
-    <link name="base_footprint"/>
+    <link name="base_footprint" />
     <joint name="base_joint" type="fixed">
-        <parent link="base_link"/>
-        <child link="base_footprint"/>
-        <origin xyz="0.0 0.0 ${-(wheel_radius+wheel_zoff)}" rpy="0 0 0"/>
+        <parent link="base_link" />
+        <child link="base_footprint" />
+        <origin xyz="0.0 0.0 ${-(wheel_radius+wheel_zoff)}" rpy="0 0 0" />
     </joint>
     <!-- Caster Wheel -->
@@ -50,27 +51,27 @@
         <visual>
             <geometry>
-                <sphere radius="${(wheel_radius+wheel_zoff-(base_height/2))}"/>
+                <sphere radius="${(wheel_radius+wheel_zoff-(base_height/2))}" />
             </geometry>
-            <material name="grey">
-                <color rgba="0.5 0.5 0.5 1.0"/>
+            <material name="gray">
+                <color rgba="0.3 0.3 0.3 1.0" />
             </material>
         </visual>
         <collision>
-            <origin xyz="0 0 0" rpy="0 0 0"/>
+            <origin xyz="0 0 0" rpy="0 0 0" />
             <geometry>
-                <sphere radius="${(wheel_radius+wheel_zoff-(base_height/2))}"/>
+                <sphere radius="${(wheel_radius+wheel_zoff-(base_height/2))}" />
             </geometry>
         </collision>
-        <xacro:sphere_inertia mass="0.5" radius="${(wheel_radius+wheel_zoff-(base_height/2))}"/>
+        <xacro:sphere_inertia mass="0.5" radius="${(wheel_radius+wheel_zoff-(base_height/2))}" />
     </link>
     <joint name="caster_joint" type="fixed">
-        <parent link="base_link"/>
-        <child link="front_caster"/>
-        <origin xyz="${caster_xoff} 0.0 ${-(base_height/2)}" rpy="0 0 0"/>
+        <parent link="base_link" />
+        <child link="front_caster" />
+        <origin xyz="${caster_xoff} 0.0 ${-(base_height/2)}" rpy="0 0 0" />
     </joint>
     <gazebo reference="front_caster">
         <material>Gazebo/Grey</material>
-        <mu1 value="0.001"/>
-        <mu2 value="0.001"/>
+        <mu1 value="0.001" />
+        <mu2 value="0.001" />
     </gazebo>
     <!-- Wheels -->

File: questbot_description/urdf/control/gazebo_control.xacro (robot description, xacro)
@@ -17,5 +17,5 @@
             <!-- output -->
             <publish_odom>true</publish_odom>
-            <publish_odom_tf>true</publish_odom_tf>
+            <publish_odom_tf>${publish_odom_tf}</publish_odom_tf>
             <publish_wheel_tf>true</publish_wheel_tf>
             <odometry_frame>odom</odometry_frame>

File: questbot_description/urdf/gazebo.urdf.xacro (robot description, xacro)
@@ -1,16 +1,20 @@
 <?xml version="1.0"?>
 <robot xmlns:xacro="http://www.ros.org/wiki/xacro">
-    <xacro:property name="use_gazebo" value="1"/>
-    <xacro:property name="use_gzsim" value="0"/>
+    <!-- Properties -->
+    <!-- Choose Gazebo version -->
+    <xacro:property name="use_gazebo" value="1" />
+    <xacro:property name="use_gzsim" value="0" />
+    <!-- Choose whether to publish odom from controller -->
+    <xacro:property name="publish_odom_tf" value="true"/>
     <!-- Classic Gazebo -->
     <xacro:if value="$(arg use_gazebo)">
         <!-- Controller -->
-        <xacro:include filename="control/gazebo_control.xacro"/>
+        <xacro:include filename="control/gazebo_control.xacro" />
         <!-- IMU gazebo plugin -->
-        <xacro:include filename="sensors/gazebo_imu.xacro"/>
+        <xacro:include filename="sensors/gazebo_imu.xacro" />
         <!-- Lidar 2D -->
-        <xacro:include filename="sensors/gazebo_lidar.xacro"/>
+        <xacro:include filename="sensors/gazebo_lidar.xacro" />
         <!-- Camera -->
-        <!-- <xacro:include filename="sensors/gazebo_camera.xacro"/> -->
+        <xacro:include filename="sensors/gazebo_camera.xacro"/>
         <!-- Depth Camera -->
         <!-- <xacro:include filename="sensors/gazebo_depth_camera.xacro"/> -->
@@ -19,5 +23,5 @@
     <xacro:if value="$(arg use_gzsim)">
         <!-- Controller -->
-        <xacro:include filename="control/gzsim_control.xacro"/>
+        <xacro:include filename="control/gzsim_control.xacro" />
     </xacro:if>
 </robot>

File: questbot_description/urdf/macro/inertial.xacro (robot description, xacro)
@@ -1,5 +1,6 @@
 <?xml version="1.0"?>
-<robot xmlns:xacro="http://www.ros.org/wiki/xacro" >
-    <!-- Specify some standard inertial calculations https://en.wikipedia.org/wiki/List_of_moments_of_inertia -->
+<robot xmlns:xacro="http://www.ros.org/wiki/xacro">
+    <!-- Specify some standard inertial calculations
+    https://en.wikipedia.org/wiki/List_of_moments_of_inertia -->
     <!-- These make use of xacro's mathematical functionality -->
     <xacro:macro name="sphere_inertia" params="mass radius">
@@ -7,6 +8,6 @@
             <mass value="${mass}" />
             <inertia ixx="${(2/5) * mass * (radius*radius)}" ixy="0.0" ixz="0.0"
-                    iyy="${(2/5) * mass * (radius*radius)}" iyz="0.0"
-                    izz="${(2/5) * mass * (radius*radius)}" />
+                iyy="${(2/5) * mass * (radius*radius)}" iyz="0.0"
+                izz="${(2/5) * mass * (radius*radius)}" />
         </inertial>
     </xacro:macro>
@@ -15,6 +16,6 @@
             <mass value="${mass}" />
             <inertia ixx="${(1/12) * mass * (height*height + length*length)}" ixy="0.0" ixz="0.0"
-                    iyy="${(1/12) * mass * (width*width +  length*length)}" iyz="0.0"
-                    izz="${(1/12) * mass * (width*width + height*height)}" />
+                iyy="${(1/12) * mass * (width*width +  length*length)}" iyz="0.0"
+                izz="${(1/12) * mass * (width*width + height*height)}" />
         </inertial>
     </xacro:macro>
@@ -23,6 +24,6 @@
             <mass value="${mass}" />
             <inertia ixx="${(1/12) * mass * (3*radius*radius + height*height)}" ixy="0.0" ixz="0.0"
-                    iyy="${(1/12) * mass * (3*radius*radius + height*height)}" iyz="0.0"
-                    izz="${(1/2) * mass * (radius*radius)}" />
+                iyy="${(1/12) * mass * (3*radius*radius + height*height)}" iyz="0.0"
+                izz="${(1/2) * mass * (radius*radius)}" />
         </inertial>
     </xacro:macro>

File: questbot_description/urdf/macro/wheel.xacro (robot description, xacro)
@@ -2,30 +2,32 @@
 <robot xmlns:xacro="http://www.ros.org/wiki/xacro">
     <!-- Include inertial macros -->
-    <xacro:include filename="inertial.xacro"/>
+    <xacro:include filename="inertial.xacro" />
     <!-- Wheels Macro -->
     <xacro:macro name="wheel" params="prefix x_reflect y_reflect">
         <link name="${prefix}_link">
             <visual>
-                <origin xyz="0 0 0" rpy="${pi/2} 0 0"/>
+                <origin xyz="0 0 0" rpy="${pi/2} 0 0" />
                 <geometry>
-                    <cylinder radius="${wheel_radius}" length="${wheel_width}"/>
+                    <cylinder radius="${wheel_radius}" length="${wheel_width}" />
                 </geometry>
-                <material name="grey">
-                    <color rgba="0.5 0.5 0.5 1.0"/>
+                <material name="gray">
+                    <color rgba="0.3 0.3 0.3 1.0" />
                 </material>
             </visual>
             <collision>
-                <origin xyz="0 0 0" rpy="${pi/2} 0 0"/>
+                <origin xyz="0 0 0" rpy="${pi/2} 0 0" />
                 <geometry>
-                <cylinder radius="${wheel_radius}" length="${wheel_width}"/>
+                    <cylinder radius="${wheel_radius}" length="${wheel_width}" />
                 </geometry>
             </collision>
-            <xacro:cyclinder_inertia mass="0.5" radius="${wheel_radius}" height="${wheel_width}"/>
+            <xacro:cyclinder_inertia mass="0.5" radius="${wheel_radius}" height="${wheel_width}" />
         </link>
         <joint name="${prefix}_joint" type="continuous">
-            <parent link="base_link"/>
-            <child link="${prefix}_link"/>
-            <origin xyz="${x_reflect*wheel_xoff} ${y_reflect*(base_width/2+wheel_ygap)} ${-wheel_zoff}" rpy="0 0 0"/>
-            <axis xyz="0 1 0"/>
+            <parent link="base_link" />
+            <child link="${prefix}_link" />
+            <origin
+                xyz="${x_reflect*wheel_xoff} ${y_reflect*(base_width/2+wheel_ygap)} ${-wheel_zoff}"
+                rpy="0 0 0" />
+            <axis xyz="0 1 0" />
         </joint>
         <gazebo reference="${prefix}_link">

File: questbot_description/urdf/robot.urdf.xacro (robot description, xacro)
@@ -2,6 +2,6 @@
 <robot xmlns:xacro="http://www.ros.org/wiki/xacro" name="questbot_2wd">
     <!-- Robot Body-->
-    <xacro:include filename="body.urdf.xacro"/>
+    <xacro:include filename="body.urdf.xacro" />
     <!-- Gazebo Definitions -->
-    <xacro:include filename="gazebo.urdf.xacro"/>
+    <xacro:include filename="gazebo.urdf.xacro" />
 </robot>

File: questbot_description/urdf/sensors/gazebo_camera.xacro (robot description, xacro)
@@ -1,25 +1,27 @@
 <?xml version="1.0"?>
-<robot xmlns:xacro="http://www.ros.org/wiki/xacro" >
+<robot xmlns:xacro="http://www.ros.org/wiki/xacro">
     <joint name="camera_joint" type="fixed">
-        <parent link="base_link"/>
-        <child link="camera_link"/>
-        <origin xyz="0.305 0 0.08" rpy="0 0 0"/>
+        <parent link="base_link" />
+        <child link="camera_link" />
+        <origin xyz="0.215 0 0.05" rpy="0 0 0" />
     </joint>
     <link name="camera_link">
         <visual>
             <geometry>
-                <box size="0.010 0.03 0.03"/>
+                <box size="0.010 0.03 0.03" />
             </geometry>
-            <material name="red"/>
+            <material name="black">
+                <color rgba="0.1 0.1 0.1 1.0" />
+            </material>
         </visual>
     </link>
     <joint name="camera_optical_joint" type="fixed">
-        <parent link="camera_link"/>
-        <child link="camera_link_optical"/>
-        <origin xyz="0 0 0" rpy="${-pi/2} 0 ${-pi/2}"/>
+        <parent link="camera_link" />
+        <child link="camera_link_optical" />
+        <origin xyz="0 0 0" rpy="${-pi/2} 0 ${-pi/2}" />
     </joint>
     <link name="camera_link_optical"></link>
     <gazebo reference="camera_link">
-        <material>Gazebo/Red</material>
+        <material>Gazebo/Black</material>
         <sensor name="camera" type="camera">
             <pose> 0 0 0 0 0 0 </pose>

File: questbot_description/urdf/sensors/gazebo_depth_camera.xacro (robot description, xacro)
@@ -3,33 +3,37 @@
     <link name="camera_link">
         <visual>
-            <origin xyz="0 0 0" rpy="0 0 0"/>
+            <origin xyz="0 0 0" rpy="0 0 0" />
             <geometry>
-            <box size="0.015 0.130 0.022"/>
+                <box size="0.015 0.130 0.022" />
             </geometry>
+            <material name="black">
+                <color rgba="0.1 0.1 0.1 1.0" />
+            </material>
         </visual>
         <collision>
-            <origin xyz="0 0 0" rpy="0 0 0"/>
+            <origin xyz="0 0 0" rpy="0 0 0" />
             <geometry>
-            <box size="0.015 0.130 0.022"/>
+                <box size="0.015 0.130 0.022" />
             </geometry>
         </collision>
         <inertial>
-            <origin xyz="0 0 0" rpy="0 0 0"/>
-            <mass value="0.035"/>
-            <inertia ixx="0.001"  ixy="0"  ixz="0" iyy="0.001" iyz="0" izz="0.001" />
+            <origin xyz="0 0 0" rpy="0 0 0" />
+            <mass value="0.035" />
+            <inertia ixx="0.001" ixy="0" ixz="0" iyy="0.001" iyz="0" izz="0.001" />
         </inertial>
     </link>
     <joint name="camera_joint" type="fixed">
-        <parent link="base_link"/>
-        <child link="camera_link"/>
-        <origin xyz="0.215 0 0.05" rpy="0 0 0"/>
+        <parent link="base_link" />
+        <child link="camera_link" />
+        <origin xyz="0.215 0 0.05" rpy="0 0 0" />
     </joint>
-    <link name="camera_depth_frame"/>
+    <link name="camera_depth_frame" />
     <joint name="camera_depth_joint" type="fixed">
-        <origin xyz="0 0 0" rpy="${-pi/2} 0 ${-pi/2}"/>
-        <parent link="camera_link"/>
-        <child link="camera_depth_frame"/>
+        <origin xyz="0 0 0" rpy="${-pi/2} 0 ${-pi/2}" />
+        <parent link="camera_link" />
+        <child link="camera_depth_frame" />
     </joint>
     <gazebo reference="camera_link">
+        <material>Gazebo/Black</material>
         <sensor name="depth_camera" type="depth">
             <visualize>true</visualize>

File: questbot_description/urdf/sensors/gazebo_imu.xacro (robot description, xacro)
@@ -1,24 +1,24 @@
 <?xml version="1.0"?>
-<robot xmlns:xacro="http://www.ros.org/wiki/xacro" >
+<robot xmlns:xacro="http://www.ros.org/wiki/xacro">
     <link name="imu_link">
         <visual>
             <geometry>
-                <box size="0.1 0.1 0.1"/>
+                <box size="0.05 0.05 0.05" />
             </geometry>
-            <material name="skyblue">
-                <color rgba="0.529 0.808 0.922 1.0"/>
+            <material name="red">
+                <color rgba="1.0 0.2 0.2 1.0" />
             </material>
         </visual>
         <collision>
             <geometry>
-                <box size="0.1 0.1 0.1"/>
+                <box size="0.1 0.1 0.1" />
             </geometry>
         </collision>
-        <xacro:box_inertia mass="0.1" width="0.1" length="0.1" height="0.1"/>
+        <xacro:box_inertia mass="0.1" width="0.1" length="0.1" height="0.1" />
     </link>
     <joint name="imu_joint" type="fixed">
-        <parent link="base_link"/>
-        <child link="imu_link"/>
-        <origin xyz="0 0 0.01"/>
+        <parent link="base_link" />
+        <child link="imu_link" />
+        <origin xyz="0 0 0.01" />
     </joint>
     <gazebo reference="imu_link">
@@ -28,64 +28,64 @@
     <gazebo reference="imu_link">
         <sensor name="imu_sensor" type="imu">
-        <plugin filename="libgazebo_ros_imu_sensor.so" name="imu_plugin">
-            <initial_orientation_as_reference>false</initial_orientation_as_reference>
-        </plugin>
-        <always_on>true</always_on>
-        <update_rate>100</update_rate>
-        <visualize>true</visualize>
-        <imu>
-            <angular_velocity>
-                <x>
-                <noise type="gaussian">
-                    <mean>0.0</mean>
-                    <stddev>2e-4</stddev>
-                    <bias_mean>0.0000075</bias_mean>
-                    <bias_stddev>0.0000008</bias_stddev>
-                </noise>
-                </x>
-                <y>
-                <noise type="gaussian">
-                    <mean>0.0</mean>
-                    <stddev>2e-4</stddev>
-                    <bias_mean>0.0000075</bias_mean>
-                    <bias_stddev>0.0000008</bias_stddev>
-                </noise>
-                </y>
-                <z>
-                <noise type="gaussian">
-                    <mean>0.0</mean>
-                    <stddev>2e-4</stddev>
-                    <bias_mean>0.0000075</bias_mean>
-                    <bias_stddev>0.0000008</bias_stddev>
-                </noise>
-                </z>
-            </angular_velocity>
-            <linear_acceleration>
-                <x>
-                <noise type="gaussian">
-                    <mean>0.0</mean>
-                    <stddev>1.7e-2</stddev>
-                    <bias_mean>0.1</bias_mean>
-                    <bias_stddev>0.001</bias_stddev>
-                </noise>
-                </x>
-                <y>
-                <noise type="gaussian">
-                    <mean>0.0</mean>
-                    <stddev>1.7e-2</stddev>
-                    <bias_mean>0.1</bias_mean>
-                    <bias_stddev>0.001</bias_stddev>
-                </noise>
-                </y>
-                <z>
-                <noise type="gaussian">
-                    <mean>0.0</mean>
-                    <stddev>1.7e-2</stddev>
-                    <bias_mean>0.1</bias_mean>
-                    <bias_stddev>0.001</bias_stddev>
-                </noise>
-                </z>
-            </linear_acceleration>
-        </imu>
+            <plugin filename="libgazebo_ros_imu_sensor.so" name="imu_plugin">
+                <initial_orientation_as_reference>false</initial_orientation_as_reference>
+            </plugin>
+            <always_on>true</always_on>
+            <update_rate>100</update_rate>
+            <visualize>true</visualize>
+            <imu>
+                <angular_velocity>
+                    <x>
+                        <noise type="gaussian">
+                            <mean>0.0</mean>
+                            <stddev>2e-4</stddev>
+                            <bias_mean>0.0000075</bias_mean>
+                            <bias_stddev>0.0000008</bias_stddev>
+                        </noise>
+                    </x>
+                    <y>
+                        <noise type="gaussian">
+                            <mean>0.0</mean>
+                            <stddev>2e-4</stddev>
+                            <bias_mean>0.0000075</bias_mean>
+                            <bias_stddev>0.0000008</bias_stddev>
+                        </noise>
+                    </y>
+                    <z>
+                        <noise type="gaussian">
+                            <mean>0.0</mean>
+                            <stddev>2e-4</stddev>
+                            <bias_mean>0.0000075</bias_mean>
+                            <bias_stddev>0.0000008</bias_stddev>
+                        </noise>
+                    </z>
+                </angular_velocity>
+                <linear_acceleration>
+                    <x>
+                        <noise type="gaussian">
+                            <mean>0.0</mean>
+                            <stddev>1.7e-2</stddev>
+                            <bias_mean>0.1</bias_mean>
+                            <bias_stddev>0.001</bias_stddev>
+                        </noise>
+                    </x>
+                    <y>
+                        <noise type="gaussian">
+                            <mean>0.0</mean>
+                            <stddev>1.7e-2</stddev>
+                            <bias_mean>0.1</bias_mean>
+                            <bias_stddev>0.001</bias_stddev>
+                        </noise>
+                    </y>
+                    <z>
+                        <noise type="gaussian">
+                            <mean>0.0</mean>
+                            <stddev>1.7e-2</stddev>
+                            <bias_mean>0.1</bias_mean>
+                            <bias_stddev>0.001</bias_stddev>
+                        </noise>
+                    </z>
+                </linear_acceleration>
+            </imu>
         </sensor>
     </gazebo>
