Commit message: linted xml & python files

File: questbot_description/urdf/sensors/gazebo_lidar.xacro (robot description, xacro)
@@ -1,29 +1,33 @@
 <?xml version="1.0"?>
-<robot xmlns:xacro="http://www.ros.org/wiki/xacro" >
+<robot xmlns:xacro="http://www.ros.org/wiki/xacro">
     <link name="lidar_link">
         <inertial>
-            <origin xyz="0 0 0" rpy="0 0 0"/>
-            <mass value="0.125"/>
-            <inertia ixx="0.001"  ixy="0"  ixz="0" iyy="0.001" iyz="0" izz="0.001" />
+            <origin xyz="0 0 0" rpy="0 0 0" />
+            <mass value="0.125" />
+            <inertia ixx="0.001" ixy="0" ixz="0" iyy="0.001" iyz="0" izz="0.001" />
         </inertial>
         <collision>
-            <origin xyz="0 0 0" rpy="0 0 0"/>
+            <origin xyz="0 0 0" rpy="0 0 0" />
             <geometry>
-            <cylinder radius="0.0508" length="0.055"/>
+                <cylinder radius="0.0508" length="0.055" />
             </geometry>
         </collision>
         <visual>
-            <origin xyz="0 0 0" rpy="0 0 0"/>
+            <origin xyz="0 0 0" rpy="0 0 0" />
             <geometry>
-            <cylinder radius="0.0508" length="0.055"/>
+                <cylinder radius="0.0508" length="0.055" />
             </geometry>
+            <material name="green">
+                <color rgba="0.0 1.0 0.0 1.0" />
+            </material>
         </visual>
     </link>
     <joint name="lidar_joint" type="fixed">
-        <parent link="base_link"/>
-        <child link="lidar_link"/>
-        <origin xyz="0 0 0.12" rpy="0 0 0"/>
+        <parent link="base_link" />
+        <child link="lidar_link" />
+        <origin xyz="0 0 0.12" rpy="0 0 0" />
     </joint>
     <gazebo reference="lidar_link">
+        <material>Gazebo/Green</material>
         <sensor name="lidar" type="ray">
             <always_on>true</always_on>
@@ -33,8 +37,8 @@
                 <scan>
                     <horizontal>
-                    <samples>360</samples>
-                    <resolution>1.000000</resolution>
-                    <min_angle>0.000000</min_angle>
-                    <max_angle>6.280000</max_angle>
+                        <samples>360</samples>
+                        <resolution>1.000000</resolution>
+                        <min_angle>0.000000</min_angle>
+                        <max_angle>6.280000</max_angle>
                     </horizontal>
                 </scan>
@@ -51,4 +55,7 @@
             </ray>
             <plugin name="scan" filename="libgazebo_ros_ray_sensor.so">
+                <ros>
+                    <remapping>~/out:=scan</remapping>
+                </ros>
                 <output_type>sensor_msgs/LaserScan</output_type>
                 <frame_name>lidar_link</frame_name>
