Commit message: restructured urdf

File: questbot_description/urdf/control/gazebo_control.xacro (robot description, xacro)
@@ -3,4 +3,7 @@
     <gazebo>
         <plugin name='diff_drive' filename='libgazebo_ros_diff_drive.so'>
+            <ros>
+                <namespace>/demo</namespace>
+            </ros>
             <!-- wheels -->
             <left_joint>left_wheel_joint</left_joint>
@@ -14,5 +17,5 @@
             <!-- output -->
             <publish_odom>true</publish_odom>
-            <publish_odom_tf>false</publish_odom_tf>
+            <publish_odom_tf>true</publish_odom_tf>
             <publish_wheel_tf>true</publish_wheel_tf>
             <odometry_frame>odom</odometry_frame>

File: questbot_description/urdf/control/gzsim_control.xacro (robot description, xacro)
@@ -3,19 +3,21 @@
   <gazebo>
     <plugin filename="gz-sim-diff-drive-system" name="gz::sim::systems::DiffDrive">
+      <ros>
+        <namespace>questbot</namespace>
+      </ros>
       <!-- Wheels -->
       <left_joint>wheel_left_joint</left_joint>
       <right_joint>wheel_right_joint</right_joint>
       <!-- Kinematics -->
-      <wheel_separation>0.35</wheel_separation>
-      <wheel_radius>0.05</wheel_radius>
+      <wheel_separation>0.4</wheel_separation>
+      <wheel_radius>0.1</wheel_radius>
       <!-- Limits -->
-      <max_linear_acceleration>10.0</max_linear_acceleration>
+      <max_acceleration>10</max_acceleration>
+      <!-- Outputs -->
       <topic>cmd_vel</topic>
-      <!-- Outputs -->
+      <!-- Odometry -->
       <odom_topic>odom</odom_topic>
       <frame_id>odom</frame_id>
       <child_frame_id>base_footprint</child_frame_id>
-      <odom_publisher_frequency>30</odom_publisher_frequency>
-      <tf_topic>/tf</tf_topic>
     </plugin>
   </gazebo>

File: questbot_description/urdf/parts/body.urdf.xacro (robot description, xacro)
@@ -2,12 +2,9 @@
 <robot xmlns:xacro="http://www.ros.org/wiki/xacro" >
     <!-- Including files -->
+    <!-- Include inertial macros -->
+    <xacro:include filename="inertial_macros.xacro"/>
+    <!-- Visual -->
     <!-- Include rviz material colors -->
     <xacro:include filename="materials.xacro"/>
-    <!-- Include gazebo material colors -->
-    <xacro:include filename="materials.gazebo.xacro"/>
-    <!-- Include inertial macros -->
-    <xacro:include filename="inertial_macro.xacro"/>
-    <!-- Include wheel macros -->
-    <xacro:include filename="wheel_macro.xacro"/>
     <!-- Define robot constants -->
     <!-- Robot base constants -->
@@ -29,5 +26,5 @@
             <box size="${base_length} ${base_width} ${base_height}"/>
         </geometry>
-        <material name="blue"/>
+        <material name="cyan"/>
         </visual>
         <collision>
@@ -66,6 +63,3 @@
         <origin xyz="${caster_xoff} 0.0 ${-(base_height/2)}" rpy="0 0 0"/>
     </joint>
-    <!-- Wheels -->
-    <xacro:wheel prefix="left_wheel" x_reflect="-1" y_reflect="1" />
-    <xacro:wheel prefix="right_wheel" x_reflect="-1" y_reflect="-1" />
 </robot>

File: questbot_description/urdf/parts/materials.xacro (robot description, xacro)
@@ -3,11 +3,17 @@
   <!-- Rviz Colours -->
   <material name="black">
-    <color rgba="0.0 0.0 0.0 1.0"/>
+    <color rgba="0 0 0 1"/>
+  </material>
+  <material name="white">
+    <color rgba="1 1 1 1"/>
   </material>
   <material name="blue">
-    <color rgba="0.0 0.0 0.8 1.0"/>
+    <color rgba="0.0 0.0 0.8 1"/>
+  </material>
+  <material name="lightblue">
+    <color rgba="0.6 0.8 1 0.9"/>
   </material>
   <material name="green">
-    <color rgba="0.0 0.8 0.0 1.0"/>
+    <color rgba="0.0 0.8 0.0 1"/>
   </material>
   <material name="grey">

File: questbot_description/urdf/parts/wheel.xacro (robot description, xacro)
@@ -1,5 +1,7 @@
 <?xml version="1.0"?>
 <robot xmlns:xacro="http://www.ros.org/wiki/xacro">
-    <!-- Wheels -->
+    <!-- Include inertial macros -->
+    <xacro:include filename="inertial_macros.xacro"/>
+    <!-- Wheels Macro -->
     <xacro:macro name="wheel" params="prefix x_reflect y_reflect">
         <link name="${prefix}_link">
@@ -26,3 +28,6 @@
         </joint>
     </xacro:macro>
+    <!-- Wheels -->
+    <xacro:wheel prefix="left_wheel" x_reflect="-1" y_reflect="1" />
+    <xacro:wheel prefix="right_wheel" x_reflect="-1" y_reflect="-1" />
 </robot>

File: questbot_description/urdf/robot.urdf.xacro (robot description, xacro)
@@ -1,19 +1,9 @@
 <?xml version="1.0"?>
-<robot xmlns:xacro="http://www.ros.org/wiki/xacro" name="robot_2wd">
-  <!-- Robot Model-->
-  <xacro:include filename="robot/robot.model.xacro"/>
-  <!-- Control Plugins -->
-  <!-- Gazebo Controller -->
-  <xacro:include filename="robot/control/gazebo_control.xacro"/>
-  <!-- Gazebo2 Controller -->
-  <!-- <xacro:include filename="questbot/control/gazebo2_control.xacro"/> -->
-  <!-- Sensor Plugins -->
-  <!-- IMU gazebo plugin -->
-  <!-- <xacro:include filename="sensors/gazebo_imu.xacro"/> -->
-  <!-- Lidar 2D -->
-  <!-- <xacro:include filename="sensors/gazebo_lidar.xacro"/> -->
-  <!-- Camera -->
-  <!-- <xacro:include filename="camera.xacro"/> -->
-  <!-- Depth Camera -->
-  <!-- <xacro:include filename="sensors/gazebo_depth_camera.xacro"/> -->
+<robot xmlns:xacro="http://www.ros.org/wiki/xacro" name="questbot_2wd">
+    <!-- Robot Body-->
+    <xacro:include filename="parts/body.urdf.xacro"/>
+    <!-- Robot Wheels -->
+    <xacro:include filename="parts/wheel.xacro"/>
+    <!-- Gazebo Definitions -->
+    <xacro:include filename="gazebo.urdf.xacro"/>
 </robot>

File: questbot_description/urdf/sensors/gazebo_imu.xacro (robot description, xacro)
@@ -6,4 +6,5 @@
                 <box size="0.1 0.1 0.1"/>
             </geometry>
+            <material name="lightblue"/>
         </visual>
         <collision>

Commit message: added changed files

File: questbot_description/urdf/control/gazebo_control.xacro (robot description, xacro)
@@ -16,4 +16,5 @@
             <max_wheel_acceleration>1.0</max_wheel_acceleration>
             <!-- output -->
+            <updateRate>100</updateRate>
             <publish_odom>true</publish_odom>
             <publish_odom_tf>${publish_odom_tf}</publish_odom_tf>

File: questbot_description/urdf/gazebo.urdf.xacro (robot description, xacro)
@@ -6,5 +6,5 @@
     <xacro:property name="use_gzsim" value="0" />
     <!-- Choose whether to publish odom from controller -->
-    <xacro:property name="publish_odom_tf" value="true"/>
+    <xacro:property name="publish_odom_tf" value="false"/>
     <!-- Classic Gazebo -->
     <xacro:if value="$(arg use_gazebo)">
